File: hitpoint/hw/Trefferzonenmodul.sch (EAGLE design)
At the start: 38 parts, among them X1 05-JST-B5B-XH-A, X2 05-JST-B5B-XH-A

Commit message: neue platine
Parts:
- removed SJ4, SJ5: (no value), jumper:SJ
- removed X1, X2: 05-JST-B5B-XH-A, con-jst-xh:05-JST-B5B-XH-A
- added +5V, 3V3, GND: (no value), wz:PINHD-1X1
- added BUS1, BUS2: 04-JST-B4B-XH-A, wz:04-JST-B4B-XH-A
- added LM1117: V_REG_MIC2920, wz:V_REG_MIC2920
- added U$5, U$6, U$7, U$8: TSOP1838, tsop:TSOP1838
- C3: value 1000µ -> (none); device rcl:C-EUC0805 -> rcl:C-EUC1210
- C4: device rcl:CPOL-EUUD-8X10 -> rcl:C-EUC1210
- R13: value 1k -> 10k
- TINY2313A: device atmel:AT90S2313S -> wz:AT90S2313S
Connections:
- removed net FREI: ULN2803.O8
- removed net LED_B1: R3.1, R6.1, ULN2803.O3
- removed net LED_B2: R12.1, R9.1, ULN2803.O6
- removed net LED_G1: R2.1, R5.1, ULN2803.O2
- removed net LED_G2: R11.1, R8.1, ULN2803.O5
- removed net LED_R1: R1.1, R4.1, ULN2803.O1
- removed net LED_R2: R10.1, R7.1, ULN2803.O4
- removed net N$20: SJ4.1, X2-4.1
- removed net N$21: SJ5.1, X1-4.1
- removed net TINY_RX: TINY2313A.(RXD)PD0, U$1.OUT, U$2.OUT, U$3.OUT, U$4.OUT
- removed net V_BATT: X1-3.1, X2-3.1
- new net +3V3: 3V3.1, C1.1, C2.1, C4.1, C6.1, C7.1, C8.1, ISP.2, LM1117.OUT, R13.1, TINY2313A.VCC, U$1.V+, U$2.V+, U$3.V+, U$4.V+, U$5.V+, U$6.V+, U$7.V+, U$8.V+
- new net FREI1: ULN2803.O1
- new net FREI5: ULN2803.O5
- new net FREI6: ULN2803.O6
- new net FREI7: ULN2803.O7
- new net LED_B: R12.1, R3.1, R6.1, R9.1, ULN2803.O4
- new net LED_G: R11.1, R2.1, R5.1, R8.1, ULN2803.O3
- new net LED_R: R1.1, R10.1, R4.1, R7.1, ULN2803.O2
- new net RX: TINY2313A.(RXD)PD0, U$1.OUT, U$2.OUT, U$3.OUT, U$4.OUT, U$5.OUT, U$6.OUT, U$7.OUT, U$8.OUT
- net +5V: now also +5V.1, BUS1-3.1, BUS2-3.1, LM1117.IN; no longer C1.1, C2.1, C4.+, C6.1, C7.1, C8.1, ISP.2, R13.1, SJ4.2, SJ5.2, TINY2313A.VCC, U$1.V+, U$2.V+, U$3.V+, U$4.V+
- net GND: now also BUS1-4.1, BUS2-4.1, C4.2, GND.1, LM1117.GND, U$5.GND, U$6.GND, U$7.GND, U$8.GND; no longer C4.-, X1-5.1, X2-5.1
- net HAPTIK: now also ULN2803.O8; no longer ULN2803.O7
- net N$1: no longer ULN2803.I1
- net N$11: now also TINY2313A.(T1/OC0B)PD5; no longer TINY2313A.(T1)PD5
- net N$3: now also TINY2313A.(OC1B)PB4; no longer TINY2313A.PB4
- net N$4: now also TINY2313A.(OC1A)PB3; no longer TINY2313A.(OCI)PB3
- net N$7: now also TINY2313A.(OC0A)PB2; no longer TINY2313A.PB2
- net SCL: now also BUS1-1.1, BUS2-1.1; no longer X1-1.1, X2-1.1
- net SDA: now also BUS1-2.1, BUS2-2.1, ULN2803.I1; no longer X1-2.1, X2-2.1
Other:
- note added: "P"
- moved on the sheet: C1, C2, C3, C6, C7, C8, ISP, R10, R11, R12, R7, R8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
