File: weapon_lasermodule/hardware/Lasermodul.brd (EAGLE design)
At the start: 51.7 x 35.5 mm, 64 parts, among them IC1 MEGA8-AI, IC2 XL6009S

Commit message: server comments
Parts:
- added C12: 100u, wz_c:C1808
- added D3: DIODE, wz:DIODE
- added L1: DR125, inductors:DR125
- added R17, R18: 10k, rcl:R0805
- C11: value (none) -> 100u; device wz:C_UNIVERSAL -> wz_c:C1808
- moved IC2 69.9 mm to (29.2, 64.1), flipped to the bottom
- moved C11 63.6 mm to (16.5, 51.4), flipped to the bottom, turned to 270 degrees
Connections:
- removed net VIN: IC2.4
- new net N$34: IC2.5, R17.1, R18.2
- new net N$36: D3.A, IC2.3, IC2.6, L1.2
- new net VCC: C11.1, IC2.4, L1.1
- net +5V: now also C12.1, D3.C, R17.2
- net GND: now also C11.2, C12.2, R18.1
Changed lines of the file:
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@@
 <element name="C4" library="wz" package="C0805" value="100n" x="36.83" y="22.225" rot="MR270"/>
 <element name="LOGO1" library="wz" package="OSHW-LOGO-M" value="OSHW-LOGOM" x="16.51" y="22.225"/>
-<element name="IC2" library="wz" package="TO263-5" value="XL6009S" x="-10.16" y="6.35"/>
-<element name="C11" library="wz" package="C_UNIVERSAL" value="" x="-12.7" y="-5.08"/>
+<element name="L1" library="inductors" package="DR125" value="DR125" x="16.51" y="65.405" rot="MR90"/>
+<element name="D3" library="wz" package="DIODE" value="DIODE" x="37.465" y="66.675" rot="MR90"/>
+<element name="C11" library="wz_c" package="C1808" value="100u" x="16.51" y="51.435" rot="MR270"/>
+<element name="C12" library="wz_c" package="C1808" value="100u" x="35.56" y="51.435" rot="MR0"/>
+<element name="R17" library="rcl" package="R0805" value="10k" x="22.225" y="57.15" rot="MR0"/>
+<element name="R18" library="rcl" package="R0805" value="10k" x="27.305" y="53.975" rot="MR0"/>
+<element name="IC2" library="wz" package="TO263-5" value="XL6009S" x="29.21" y="64.135" rot="MR0"/>
 </elements>
 <signals>
@@
 <wire x1="45.72" y1="4.445" x2="45.72" y2="12.065" width="1.27" layer="16"/>
 <wire x1="45.72" y1="12.065" x2="45.72" y2="22.225" width="1.27" layer="16"/>
+<contactref element="D3" pad="C"/>
+<contactref element="C12" pad="1"/>
+<contactref element="R17" pad="2"/>
+<wire x1="37.764" y1="51.435" x2="37.465" y2="64.475" width="0" layer="19" extent="16-16"/>
+<wire x1="21.275" y1="57.15" x2="37.764" y2="51.435" width="0" layer="19" extent="16-16"/>
+<wire x1="35.56" y1="33.02" x2="37.764" y2="51.435" width="0" layer="19" extent="16-16"/>
 </signal>
 <signal name="GND">
@@
 <vertex x="22.225" y="7.62"/>
 </polygon>
+<contactref element="C11" pad="2"/>
+<contactref element="R18" pad="1"/>
+<contactref element="C12" pad="2"/>
 <contactref element="IC2" pad="1"/>
-<wire x1="40.64" y1="22.225" x2="48.26" y2="22.225" width="0" layer="19" extent="1-1"/>
-<wire x1="38.735" y1="21.1988" x2="40.64" y2="22.225" width="0" layer="19" extent="16-16"/>
+<wire x1="28.255" y1="53.975" x2="32.6136" y2="58.3438" width="0" layer="19" extent="16-16"/>
+<wire x1="33.356" y1="51.435" x2="28.255" y2="53.975" width="0" layer="19" extent="16-16"/>
+<wire x1="16.51" y1="49.231" x2="28.255" y2="53.975" width="0" layer="19" extent="16-16"/>
+<wire x1="20.419" y1="30.33" x2="16.51" y2="49.231" width="0" layer="19" extent="16-16"/>
+<wire x1="24.701" y1="29.06" x2="20.419" y2="30.33" width="0" layer="19" extent="16-16"/>
+<wire x1="21.493528125" y1="25.24983125" x2="24.701" y2="29.06" width="0" layer="19" extent="16-16"/>
+<wire x1="29.845" y1="24.765" x2="24.701" y2="29.06" width="0" layer="19" extent="16-16"/>
+<wire x1="32.15" y1="19.5326" x2="29.845" y2="24.765" width="0" layer="19" extent="16-16"/>
+<wire x1="36.83" y1="21.1988" x2="32.15" y2="19.5326" width="0" layer="19" extent="16-16"/>
+<wire x1="38.735" y1="21.1988" x2="36.83" y2="21.1988" width="0" layer="19" extent="16-16"/>
 <wire x1="38.1" y1="19.7587" x2="38.735" y2="21.1988" width="0" layer="19" extent="16-16"/>
 <wire x1="40.005" y1="19.7587" x2="38.1" y2="19.7587" width="0" layer="19" extent="16-16"/>
-<wire x1="36.83" y1="21.1988" x2="38.735" y2="21.1988" width="0" layer="19" extent="16-16"/>
-<wire x1="32.15" y1="19.5326" x2="36.83" y2="21.1988" width="0" layer="19" extent="16-16"/>
+<wire x1="40.64" y1="22.225" x2="38.735" y2="21.1988" width="0" layer="19" extent="16-16"/>
 <wire x1="42.175" y1="14.9225" x2="40.005" y2="19.7587" width="0" layer="19" extent="16-16"/>
-<wire x1="29.845" y1="24.765" x2="32.15" y2="19.5326" width="0" layer="19" extent="16-16"/>
 <wire x1="35.0012" y1="27.5336" x2="29.845" y2="24.765" width="0" layer="19" extent="16-16"/>
-<wire x1="24.701" y1="29.06" x2="29.845" y2="24.765" width="0" layer="19" extent="16-16"/>
-<wire x1="20.419" y1="30.33" x2="24.701" y2="29.06" width="0" layer="19" extent="16-16"/>
-<wire x1="21.493528125" y1="25.24983125" x2="24.701" y2="29.06" width="0" layer="19" extent="16-16"/>
 <wire x1="48.26" y1="12.065" x2="42.175" y2="14.9225" width="0" layer="19" extent="16-16"/>
+<wire x1="48.26" y1="22.225" x2="40.64" y2="22.225" width="0" layer="19" extent="1-1"/>
 <wire x1="48.26" y1="4.445" x2="48.26" y2="12.065" width="0" layer="19" extent="1-1"/>
 <wire x1="31.35" y1="10.9474" x2="32.15" y2="19.5326" width="0" layer="19" extent="16-16"/>
@@
 <wire x1="2.1488" y1="20.32" x2="2.1488" y2="17.78" width="0" layer="19" extent="16-16"/>
 <wire x1="2.1488" y1="22.86" x2="2.1488" y2="20.32" width="0" layer="19" extent="16-16"/>
-<wire x1="-13.5636" y1="0.5588" x2="2.1488" y2="7.62" width="0" layer="19" extent="1-16"/>
 </signal>
 <signal name="V_BATT">
@@
 </polygon>
 </signal>
-<signal name="VIN">
+<signal name="N$34">
+<contactref element="R17" pad="1"/>
+<contactref element="R18" pad="2"/>
+<contactref element="IC2" pad="5"/>
+<wire x1="23.175" y1="57.15" x2="25.8064" y2="58.3438" width="0" layer="19" extent="16-16"/>
+<wire x1="26.355" y1="53.975" x2="25.8064" y2="58.3438" width="0" layer="19" extent="16-16"/>
+</signal>
+<signal name="N$36">
+<contactref element="D3" pad="A"/>
+<contactref element="L1" pad="2"/>
+<contactref element="IC2" pad="6"/>
+<contactref element="IC2" pad="3"/>
+<wire x1="29.21" y1="66.675" x2="37.465" y2="68.875" width="0" layer="19" extent="16-16"/>
+<wire x1="29.21" y1="58.3438" x2="29.21" y2="66.675" width="0" layer="19" extent="16-16"/>
+<wire x1="16.51" y1="70.38" x2="29.21" y2="66.675" width="0" layer="19" extent="16-16"/>
+</signal>
+<signal name="VCC">
+<contactref element="C11" pad="1"/>
+<contactref element="L1" pad="1"/>
 <contactref element="IC2" pad="4"/>
+<wire x1="16.51" y1="60.43" x2="27.5082" y2="58.3438" width="0" layer="19" extent="16-16"/>
+<wire x1="16.51" y1="53.639" x2="16.51" y2="60.43" width="0" layer="19" extent="16-16"/>
 </signal>
 </signals>
