File: hitpoint/hardware/Trefferzonenmodul.brd (EAGLE design)
At the start: 53.3 x 53.3 mm, 43 parts

Commit message: hitpoint hardware, touch
hitpoint: sda ist nun nicht mehr mit dem uln verbunden, pegel nun 3,3v
statt 2,5v
touch in x lauffähig
oszi messungen am i2s hinzugefügt
Parts:
- TINY2313A: value AT90S2313S -> TINY2313A; device wz:SO20L -> wz:SO20LVERSTUMMELT
Connections:
- net SDA: no longer ULN2803.1
Routing:
- net SDA: track 39.4 -> 37.2 mm
Changed lines of the file:
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@@
 <layer number="223" name="223bmp" color="24" fill="1" visible="no" active="no"/>
 <layer number="224" name="224bmp" color="25" fill="1" visible="no" active="no"/>
+<layer number="231" name="Eagle3D_PG1" color="7" fill="1" visible="yes" active="yes"/>
+<layer number="232" name="Eagle3D_PG2" color="7" fill="1" visible="yes" active="yes"/>
+<layer number="233" name="Eagle3D_PG3" color="7" fill="1" visible="yes" active="yes"/>
 <layer number="248" name="Housing" color="7" fill="1" visible="yes" active="yes"/>
 <layer number="249" name="Edge" color="7" fill="1" visible="yes" active="yes"/>
@@
 </autorouter>
 <elements>
-<element name="TINY2313A" library="wz" package="SO20L" value="AT90S2313S" x="29.21" y="23.495" rot="MR270">
-<attribute name="OC_NEWARK" value="unknown" x="35.56" y="-0.635" size="1.778" layer="28" rot="MR270" display="off"/>
-<attribute name="MPN" value="" x="35.56" y="-0.635" size="1.778" layer="28" rot="MR270" display="off"/>
-<attribute name="MF" value="" x="35.56" y="-0.635" size="1.778" layer="28" rot="MR270" display="off"/>
-<attribute name="OC_FARNELL" value="unknown" x="35.56" y="-0.635" size="1.778" layer="28" rot="MR270" display="off"/>
-</element>
+<element name="TINY2313A" library="wz" package="SO20LVERSTUMMELT" value="TINY2313A" x="29.21" y="23.495" rot="MR270"/>
 <element name="C1" library="wz" package="C0805" value="100n" x="21.355" y="26.77" rot="MR0"/>
 <element name="R1" library="wz" package="R0805" value="100" x="30.48" y="8.89" rot="MR270"/>
@@
 <contactref element="TINY2313A" pad="17"/>
 <contactref element="ISP" pad="4"/>
-<contactref element="ULN2803" pad="1"/>
-<wire x1="22.8092" y1="24.765" x2="24.8158" y2="24.765" width="0.4064" layer="16"/>
 <wire x1="25.4" y1="31.4325" x2="27.94" y2="28.8925" width="0.4064" layer="16"/>
 <wire x1="27.94" y1="28.8925" x2="27.94" y2="26.67" width="0.4064" layer="16"/>
 <wire x1="27.94" y1="26.67" x2="26.035" y2="24.765" width="0.4064" layer="16"/>
-<wire x1="26.035" y1="24.765" x2="24.8158" y2="24.765" width="0.4064" layer="16"/>
+<wire x1="26.035" y1="24.765" x2="25.0698" y2="24.765" width="0.4064" layer="16"/>
 <wire x1="15.24" y1="29.845" x2="15.875" y2="29.845" width="0.4064" layer="16"/>
 <wire x1="15.875" y1="29.845" x2="17.145" y2="31.115" width="0.4064" layer="16"/>
