File: hitpoint/hardware/hitpoint.brd (EAGLE design)
At the start: 49.5 x 49.5 mm, 47 parts

Commit message: routing
Other:
- board text added: "C3"
- board text added: "Lasertag Hitpoint v1.1 warpzone.ms"
- board text removed: "Lasertag Hitpoint v1.0 warpzone.ms"
