File: lasermodule/hardware/ansatz mit diskret step up/Lasermodul.brd (EAGLE design)
At the start: 51.7 x 35.5 mm, 67 parts, among them IC1 MEGA8-AI

Commit message: i2c
Parts:
- removed DISPLAY: (no value), con-lstb:MA12-1
- removed PI: (no value), con-lstb:MA13-2
- removed U$2: (no value), wz:PI2
- removed U$3: XL6009-STEPUP-BOARD, wz:XL6009-STEPUP-BOARD
- removed U$4: PAM8403-AMP-BOARD, wz:PAM8403-AMP-BOARD
- added C11, C12: 100u, wz_c:C1808
- added D3: DIODE, wz:DIODE
- added IC2: XL6009S, wz:TO263-5
- added L1: DR125, inductors:DR125
- added R17, R18: 10k, rcl:R0805
Connections:
- removed net OUT+: U$3.OUT+
- removed net PGND: U$4.PGND
- new net N$34: IC2.5, R17.1, R18.2
- new net N$36: D3.A, IC2.3, IC2.6, L1.2
- net +5V: now also C12.1, D3.C, R17.2
- net GND: now also C11.2, C12.2, IC2.1, R18.1; no longer U$3.GND_IN, U$3.GND_OUT
- net VCC: now also C11.1, IC2.4, L1.1; no longer U$4.VCC
Changed lines of the file:
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@@
 <wire x1="51.74" y1="35.55" x2="0" y2="35.55" width="0.4064" layer="20"/>
 <wire x1="0" y1="35.55" x2="0" y2="0" width="0.4064" layer="20"/>
-<dimension x1="0" y1="0" x2="100.33" y2="0" x3="50.165" y3="0" textsize="1.778" layer="16"/>
-<dimension x1="0" y1="0" x2="0" y2="80.01" x3="0" y3="40.005" textsize="1.778" layer="16"/>
-<dimension x1="99.695" y1="0" x2="99.695" y2="80.01" x3="100.33" y3="40.005" textsize="1.778" layer="16"/>
-<dimension x1="0" y1="80.01" x2="100.33" y2="80.01" x3="50.165" y3="80.01" textsize="1.778" layer="16"/>
 </plain>
 <attributes>
@@
 <element name="C4" library="wz" package="C0805" value="100n" x="36.83" y="22.225" rot="MR270"/>
 <element name="LOGO1" library="wz" package="OSHW-LOGO-M" value="OSHW-LOGOM" x="16.51" y="22.225"/>
-<element name="U$3" library="wz" package="XL6009-STEPUP-BOARD" value="XL6009-STEPUP-BOARD" x="5.08" y="48.895"/>
-<element name="U$4" library="wz" package="PAM8403-AMP-BOARD" value="PAM8403-AMP-BOARD" x="62.23" y="38.1"/>
-<element name="PI" library="con-lstb" package="MA13-2" value="" x="29.21" y="78.105">
-<attribute name="OC_NEWARK" value="unknown" x="29.21" y="78.105" size="1.778" layer="27" display="off"/>
-<attribute name="MPN" value="" x="29.21" y="78.105" size="1.778" layer="27" display="off"/>
-<attribute name="MF" value="" x="29.21" y="78.105" size="1.778" layer="27" display="off"/>
-<attribute name="OC_FARNELL" value="unknown" x="29.21" y="78.105" size="1.778" layer="27" display="off"/>
-</element>
-<element name="U$2" library="wz" package="PI2" value="" x="147.32" y="51.435"/>
-<element name="DISPLAY" library="con-lstb" package="MA12-1" value="" x="13.335" y="-23.495">
-<attribute name="OC_NEWARK" value="unknown" x="13.335" y="-23.495" size="1.778" layer="27" display="off"/>
-<attribute name="MPN" value="" x="13.335" y="-23.495" size="1.778" layer="27" display="off"/>
-<attribute name="MF" value="" x="13.335" y="-23.495" size="1.778" layer="27" display="off"/>
-<attribute name="OC_FARNELL" value="unknown" x="13.335" y="-23.495" size="1.778" layer="27" display="off"/>
-</element>
+<element name="L1" library="inductors" package="DR125" value="DR125" x="16.51" y="65.405" rot="MR90"/>
+<element name="D3" library="wz" package="DIODE" value="DIODE" x="37.465" y="66.675" rot="MR90"/>
+<element name="C11" library="wz_c" package="C1808" value="100u" x="16.51" y="51.435" rot="MR270"/>
+<element name="C12" library="wz_c" package="C1808" value="100u" x="35.56" y="51.435" rot="MR0"/>
+<element name="R17" library="rcl" package="R0805" value="10k" x="22.225" y="57.15" rot="MR0"/>
+<element name="R18" library="rcl" package="R0805" value="10k" x="27.305" y="53.975" rot="MR0"/>
+<element name="IC2" library="wz" package="TO263-5" value="XL6009S" x="29.21" y="64.135" rot="MR0"/>
 </elements>
 <signals>
@@
 <wire x1="45.72" y1="4.445" x2="45.72" y2="12.065" width="1.27" layer="16"/>
 <wire x1="45.72" y1="12.065" x2="45.72" y2="22.225" width="1.27" layer="16"/>
+<contactref element="D3" pad="C"/>
+<contactref element="C12" pad="1"/>
+<contactref element="R17" pad="2"/>
+<wire x1="37.764" y1="51.435" x2="37.465" y2="64.475" width="0" layer="19" extent="16-16"/>
+<wire x1="21.275" y1="57.15" x2="37.764" y2="51.435" width="0" layer="19" extent="16-16"/>
+<wire x1="35.56" y1="33.02" x2="37.764" y2="51.435" width="0" layer="19" extent="16-16"/>
 </signal>
 <signal name="GND">
@@
 <vertex x="22.225" y="7.62"/>
 </polygon>
-<contactref element="U$3" pad="GND_IN"/>
-<contactref element="U$3" pad="GND_OUT"/>
-<wire x1="6.88" y1="68.095" x2="46.28" y2="68.095" width="0" layer="19" extent="1-1"/>
-<wire x1="20.419" y1="30.33" x2="6.88" y2="68.095" width="0" layer="19" extent="16-16"/>
+<contactref element="C11" pad="2"/>
+<contactref element="R18" pad="1"/>
+<contactref element="C12" pad="2"/>
+<contactref element="IC2" pad="1"/>
+<wire x1="28.255" y1="53.975" x2="32.6136" y2="58.3438" width="0" layer="19" extent="16-16"/>
+<wire x1="33.356" y1="51.435" x2="28.255" y2="53.975" width="0" layer="19" extent="16-16"/>
+<wire x1="16.51" y1="49.231" x2="28.255" y2="53.975" width="0" layer="19" extent="16-16"/>
+<wire x1="20.419" y1="30.33" x2="16.51" y2="49.231" width="0" layer="19" extent="16-16"/>
 <wire x1="24.701" y1="29.06" x2="20.419" y2="30.33" width="0" layer="19" extent="16-16"/>
 <wire x1="21.493528125" y1="25.24983125" x2="24.701" y2="29.06" width="0" layer="19" extent="16-16"/>
@@
 </polygon>
 </signal>
-<signal name="OUT-">
-</signal>
-<signal name="OUT+">
-<contactref element="U$3" pad="OUT+"/>
+<signal name="N$34">
+<contactref element="R17" pad="1"/>
+<contactref element="R18" pad="2"/>
+<contactref element="IC2" pad="5"/>
+<wire x1="23.175" y1="57.15" x2="25.8064" y2="58.3438" width="0" layer="19" extent="16-16"/>
+<wire x1="26.355" y1="53.975" x2="25.8064" y2="58.3438" width="0" layer="19" extent="16-16"/>
+</signal>
+<signal name="N$36">
+<contactref element="D3" pad="A"/>
+<contactref element="L1" pad="2"/>
+<contactref element="IC2" pad="6"/>
+<contactref element="IC2" pad="3"/>
+<wire x1="29.21" y1="66.675" x2="37.465" y2="68.875" width="0" layer="19" extent="16-16"/>
+<wire x1="29.21" y1="58.3438" x2="29.21" y2="66.675" width="0" layer="19" extent="16-16"/>
+<wire x1="16.51" y1="70.38" x2="29.21" y2="66.675" width="0" layer="19" extent="16-16"/>
 </signal>
 <signal name="VCC">
-<contactref element="U$4" pad="VCC"/>
-</signal>
-<signal name="PGND">
-<contactref element="U$4" pad="PGND"/>
+<contactref element="C11" pad="1"/>
+<contactref element="L1" pad="1"/>
+<contactref element="IC2" pad="4"/>
+<wire x1="16.51" y1="60.43" x2="27.5082" y2="58.3438" width="0" layer="19" extent="16-16"/>
+<wire x1="16.51" y1="53.639" x2="16.51" y2="60.43" width="0" layer="19" extent="16-16"/>
 </signal>
 </signals>
