File: lasermodule/hardware/ansatz mit diskret step up/Lasermodul.sch (EAGLE design)
At the start: 66 parts, among them IC1 MEGA8-AI

Commit message: i2c
Parts:
- removed DISPLAY: (no value), con-lstb:MA12-1
- removed PI: (no value), con-lstb:MA13-2
- removed U$3: XL6009-STEPUP-BOARD, wz:XL6009-STEPUP-BOARD
- removed U$4: PAM8403-AMP-BOARD, wz:PAM8403-AMP-BOARD
- added C11, C12: 100u, wz_c:C-EUC1808
- added D3: DIODE, wz:DIODE
- added IC2: XL6009S, wz:XL6009S
- added L1: DR125, inductors:DR125
- added R17, R18: 10k, rcl:R-EU_R0805
Connections:
- new net N$34: IC2.FB, R17.1, R18.2
- new net N$36: D3.A, IC2.SW, L1.2
- new net VCC: C11.1, IC2.VIN, L1.1
- net +5V: now also C12.1, D3.C, R17.2
- net GND: now also C11.2, C12.2, IC2.GND, R18.1
Changed lines of the file:
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@@
 <part name="C4" library="wz" deviceset="C-EU" device="C0805" value="100n"/>
 <part name="LOGO1" library="wz" deviceset="OSHW-LOGO" device="M"/>
-<part name="U$3" library="wz" deviceset="XL6009-STEPUP-BOARD" device=""/>
-<part name="U$4" library="wz" deviceset="PAM8403-AMP-BOARD" device=""/>
-<part name="PI" library="con-lstb" deviceset="MA13-2" device=""/>
-<part name="DISPLAY" library="con-lstb" deviceset="MA12-1" device=""/>
+<part name="L1" library="inductors" deviceset="DR125" device=""/>
+<part name="D3" library="wz" deviceset="DIODE" device=""/>
+<part name="C11" library="wz_c" deviceset="C-EU" device="C1808" value="100u"/>
+<part name="C12" library="wz_c" deviceset="C-EU" device="C1808" value="100u"/>
+<part name="GND14" library="supply1" deviceset="GND" device=""/>
+<part name="P+3" library="supply1" deviceset="+5V" device=""/>
+<part name="P+4" library="supply1" deviceset="VCC" device="" value="VCC"/>
+<part name="R17" library="rcl" deviceset="R-EU_" device="R0805" value="10k"/>
+<part name="R18" library="rcl" deviceset="R-EU_" device="R0805" value="10k"/>
+<part name="IC2" library="wz" deviceset="XL6009" device="S"/>
 </parts>
 <sheets>
@@
 <instance part="C4" gate="G$1" x="101.6" y="58.42"/>
 <instance part="LOGO1" gate="G$1" x="116.84" y="106.68"/>
-<instance part="U$3" gate="G$1" x="35.56" y="-63.5"/>
-<instance part="U$4" gate="G$1" x="76.2" y="-73.66"/>
-<instance part="PI" gate="G$1" x="-12.7" y="-63.5" rot="R270"/>
-<instance part="DISPLAY" gate="1" x="-20.32" y="-25.4"/>
+<instance part="L1" gate="G$1" x="15.24" y="-55.88"/>
+<instance part="D3" gate="G$1" x="30.48" y="-55.88"/>
+<instance part="C11" gate="G$1" x="-12.7" y="-73.66"/>
+<instance part="C12" gate="G$1" x="55.88" y="-71.12"/>
+<instance part="GND14" gate="1" x="-12.7" y="-91.44"/>
+<instance part="P+3" gate="1" x="60.96" y="-53.34"/>
+<instance part="P+4" gate="VCC" x="-12.7" y="-63.5"/>
+<instance part="R17" gate="G$1" x="43.18" y="-68.58" rot="R90"/>
+<instance part="R18" gate="G$1" x="43.18" y="-83.82" rot="R90"/>
+<instance part="IC2" gate="A" x="20.32" y="-73.66"/>
 </instances>
 <busses>
@@
 <wire x1="144.78" y1="-53.34" x2="142.24" y2="-53.34" width="0.1524" layer="91"/>
 <label x="144.78" y="-53.34" size="1.778" layer="95"/>
+</segment>
+<segment>
+<pinref part="R17" gate="G$1" pin="2"/>
+<wire x1="43.18" y1="-63.5" x2="43.18" y2="-55.88" width="0.1524" layer="91"/>
+<pinref part="D3" gate="G$1" pin="C"/>
+<wire x1="43.18" y1="-55.88" x2="33.02" y2="-55.88" width="0.1524" layer="91"/>
+<pinref part="C12" gate="G$1" pin="1"/>
+<wire x1="55.88" y1="-68.58" x2="55.88" y2="-55.88" width="0.1524" layer="91"/>
+<wire x1="55.88" y1="-55.88" x2="43.18" y2="-55.88" width="0.1524" layer="91"/>
+<pinref part="P+3" gate="1" pin="+5V"/>
+<wire x1="60.96" y1="-55.88" x2="55.88" y2="-55.88" width="0.1524" layer="91"/>
 </segment>
 </net>
@@
 <wire x1="144.78" y1="-55.88" x2="142.24" y2="-55.88" width="0.1524" layer="91"/>
 <label x="144.78" y="-55.88" size="1.778" layer="95"/>
+</segment>
+<segment>
+<pinref part="C11" gate="G$1" pin="2"/>
+<pinref part="GND14" gate="1" pin="GND"/>
+<wire x1="-12.7" y1="-78.74" x2="-12.7" y2="-88.9" width="0.1524" layer="91"/>
+<wire x1="-12.7" y1="-88.9" x2="33.02" y2="-88.9" width="0.1524" layer="91"/>
+<wire x1="33.02" y1="-88.9" x2="33.02" y2="-78.74" width="0.1524" layer="91"/>
+<pinref part="R18" gate="G$1" pin="1"/>
+<wire x1="33.02" y1="-88.9" x2="43.18" y2="-88.9" width="0.1524" layer="91"/>
+<pinref part="C12" gate="G$1" pin="2"/>
+<wire x1="43.18" y1="-88.9" x2="55.88" y2="-88.9" width="0.1524" layer="91"/>
+<wire x1="55.88" y1="-88.9" x2="55.88" y2="-76.2" width="0.1524" layer="91"/>
+<junction x="33.02" y="-88.9"/>
+<pinref part="IC2" gate="A" pin="GND"/>
 </segment>
 </net>
@@
 </segment>
 </net>
+<net name="N$34" class="0">
+<segment>
+<pinref part="R17" gate="G$1" pin="1"/>
+<pinref part="R18" gate="G$1" pin="2"/>
+<wire x1="43.18" y1="-73.66" x2="43.18" y2="-78.74" width="0.1524" layer="91"/>
+<wire x1="43.18" y1="-73.66" x2="33.02" y2="-73.66" width="0.1524" layer="91"/>
+<junction x="43.18" y="-73.66"/>
+<pinref part="IC2" gate="A" pin="FB"/>
+</segment>
+</net>
+<net name="N$36" class="0">
+<segment>
+<pinref part="D3" gate="G$1" pin="A"/>
+<pinref part="L1" gate="G$1" pin="2"/>
+<wire x1="27.94" y1="-55.88" x2="25.4" y2="-55.88" width="0.1524" layer="91"/>
+<wire x1="25.4" y1="-55.88" x2="22.86" y2="-55.88" width="0.1524" layer="91"/>
+<wire x1="33.02" y1="-68.58" x2="33.02" y2="-63.5" width="0.1524" layer="91"/>
+<wire x1="33.02" y1="-63.5" x2="25.4" y2="-63.5" width="0.1524" layer="91"/>
+<wire x1="25.4" y1="-63.5" x2="25.4" y2="-55.88" width="0.1524" layer="91"/>
+<junction x="25.4" y="-55.88"/>
+<pinref part="IC2" gate="A" pin="SW"/>
+</segment>
+</net>
+<net name="VCC" class="0">
+<segment>
+<pinref part="P+4" gate="VCC" pin="VCC"/>
+<pinref part="C11" gate="G$1" pin="1"/>
+<wire x1="-12.7" y1="-66.04" x2="-12.7" y2="-68.58" width="0.1524" layer="91"/>
+<wire x1="-12.7" y1="-71.12" x2="-12.7" y2="-68.58" width="0.1524" layer="91"/>
+<pinref part="L1" gate="G$1" pin="1"/>
+<wire x1="7.62" y1="-55.88" x2="7.62" y2="-68.58" width="0.1524" layer="91"/>
+<wire x1="7.62" y1="-68.58" x2="10.16" y2="-68.58" width="0.1524" layer="91"/>
+<wire x1="-12.7" y1="-68.58" x2="7.62" y2="-68.58" width="0.1524" layer="91"/>
+<junction x="-12.7" y="-68.58"/>
+<junction x="7.62" y="-68.58"/>
+<pinref part="IC2" gate="A" pin="VIN"/>
+</segment>
+</net>
 </nets>
 </sheet>
@@
 </schematic>
 </drawing>
-<compatibility>
-<note version="6.3" minversion="6.2.2" severity="warning">
-Since Version 6.2.2 text objects can contain more than one line,
-which will not be processed correctly with this version.
-</note>
-</compatibility>
 </eagle>
