File: lasermodule/hardware/Lasermodul.brd (EAGLE design)
At the start: 51.7 x 35.5 mm, 67 parts, among them IC1 MEGA8-AI

Commit message: the real real Hitpoint 1.0
so wurden die ersten 20 platinen bestellt
Parts:
- added K3G1, K3G2, K3G3, K3G4, K3G5, K3G6: (no value), wz:PIN-HEADER-1
- +5V, B+, B-, GND, I+, I-, K1, K1G, K2, K2G, K3, K3G, L+1, L+2, L+3, LB, LG, LR, T5V, TB, TG, TR, TW: device wz:1X01 -> wz:PIN-HEADER-1
- BUS, ZUM_PI: value 04-JST-B4B-XH-A -> JST-XH_BUCHSE-4-; device wz:B4B-XH -> wz:JST-XH_BUCHSE-4
- C1, C4, C5: device wz:C0805 -> wz:0603
- C10, C7, C8, C9: device wz:C0805 -> wz:0805
- C2: value 100u -> 4.7u; device wz_c:C1808 -> wz:0805
- C3: value 100u -> 1000u; device wz_c:C1808 -> wz:C_UNIVERSAL
- C6: device rcl:C0805 -> wz:0603
- D1: device wz:F126Z12 -> wz:Z-DIODE
- LM1117: value V_REG_MIC2920 -> LM1117_3V3_REGULATOR
- R1, R10, R11, R12, R13, R14, R15, R2, R3, R6, R7, R8, R9: device rcl:R0805 -> wz:0603
- R16, R4, R5: device wz:R0805 -> wz:0603
- moved U$2 88.7 mm to (80.0, -6.35)
- moved U$3 68.8 mm to (73.7, 43.8), turned to 180 degrees
- moved DISPLAY 62.3 mm to (15.2, 38.7)
- moved U$4 41.8 mm to (81.9, 1.27), turned to 180 degrees
- moved PI 33.8 mm to (18.4, 46.1)
Connections:
- removed net OUT+: U$3.OUT+
- removed net PGND: U$4.PGND
- removed net VCC: U$4.VCC
- new net N$34: K3G3.1, U$3.IN+
- net +5V: now also C3.1B, K3G1.1, K3G6.1, U$3.OUT+, U$4.VCC
- net GND: now also C3.2B, K3G2.1, K3G4.1, K3G5.1, U$4.AGND, U$4.PGND

Commit message: laserbodul hardware weiter gemacht
umstellung auf pi modul mit fast allem drauf
Parts:
- added AMP_IN_L, AMP_IN_R, AMP_OUT_L_+, AMP_OUT_L_-, AMP_OUT_R_+, AMP_OUT_R_-: (no value), wz:PIN-HEADER-1
- renumbered K3G1 to AMP_5V, K3G2 to AMP_GND, K3G3 to LIPO+, K3G4 to LIPO-, K3G5 to MISC_GND, K3G6 to MISC_5V
Connections:
- new net N$35: AMP_IN_L.1, U$4.IN_L
- new net N$36: AMP_IN_R.1, U$4.IN_R
- new net N$37: AMP_OUT_L_+.1, U$4.OUT_L_+
- new net N$38: AMP_OUT_L_-.1, U$4.OUT_L_-
- new net N$39: AMP_OUT_R_-.1, U$4.OUT_R_-
- new net N$40: AMP_OUT_R_+.1, U$4.OUT_R_+
Changed lines of the file:
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@@
 <attribute name="OC_FARNELL" value="unknown" x="15.24" y="38.735" size="1.778" layer="27" display="off"/>
 </element>
-<element name="K3G1" library="wz" package="PIN-HEADER-1" value="" x="-0.635" y="-30.48"/>
-<element name="K3G2" library="wz" package="PIN-HEADER-1" value="" x="-0.635" y="-36.195"/>
+<element name="AMP_5V" library="wz" package="PIN-HEADER-1" value="" x="-0.635" y="-30.48"/>
+<element name="AMP_GND" library="wz" package="PIN-HEADER-1" value="" x="-0.635" y="-36.195"/>
 <element name="U$4" library="wz" package="PAM8403-AMP-BOARD" value="PAM8403-AMP-BOARD" x="81.915" y="1.27" rot="R180"/>
-<element name="K3G3" library="wz" package="PIN-HEADER-1" value="" x="-31.115" y="-41.91"/>
-<element name="K3G4" library="wz" package="PIN-HEADER-1" value="" x="-31.115" y="-47.625"/>
-<element name="K3G5" library="wz" package="PIN-HEADER-1" value="" x="-31.115" y="-53.34"/>
-<element name="K3G6" library="wz" package="PIN-HEADER-1" value="" x="-31.115" y="-59.055"/>
+<element name="LIPO+" library="wz" package="PIN-HEADER-1" value="" x="-31.115" y="-41.91"/>
+<element name="LIPO-" library="wz" package="PIN-HEADER-1" value="" x="-31.115" y="-47.625"/>
+<element name="MISC_GND" library="wz" package="PIN-HEADER-1" value="" x="-31.115" y="-53.34"/>
+<element name="MISC_5V" library="wz" package="PIN-HEADER-1" value="" x="-31.115" y="-59.055"/>
+<element name="AMP_IN_L" library="wz" package="PIN-HEADER-1" value="" x="-31.115" y="-64.77"/>
+<element name="AMP_IN_R" library="wz" package="PIN-HEADER-1" value="" x="-31.115" y="-70.485"/>
+<element name="AMP_OUT_L_-" library="wz" package="PIN-HEADER-1" value="" x="-31.115" y="-76.2"/>
+<element name="AMP_OUT_L_+" library="wz" package="PIN-HEADER-1" value="" x="-31.115" y="-81.915"/>
+<element name="AMP_OUT_R_-" library="wz" package="PIN-HEADER-1" value="" x="-31.115" y="-87.63"/>
+<element name="AMP_OUT_R_+" library="wz" package="PIN-HEADER-1" value="" x="-31.115" y="-93.345"/>
 </elements>
 <signals>
@@
 <contactref element="U$3" pad="OUT+"/>
 <contactref element="U$4" pad="VCC"/>
-<contactref element="K3G1" pad="1"/>
-<contactref element="K3G6" pad="1"/>
+<contactref element="AMP_5V" pad="1"/>
+<contactref element="MISC_5V" pad="1"/>
 <wire x1="49.53" y1="33.02" x2="71.86" y2="42.015" width="0" layer="19" extent="16-16"/>
 <wire x1="15.675" y1="30.33" x2="15.725" y2="30.33" width="0" layer="19" extent="16-16"/>
@@
 <contactref element="U$4" pad="AGND"/>
 <contactref element="U$4" pad="PGND"/>
-<contactref element="K3G2" pad="1"/>
-<contactref element="K3G4" pad="1"/>
-<contactref element="K3G5" pad="1"/>
+<contactref element="AMP_GND" pad="1"/>
+<contactref element="LIPO-" pad="1"/>
+<contactref element="MISC_GND" pad="1"/>
 <wire x1="67.945" y1="2.54" x2="71.86" y2="24.615" width="0" layer="19" extent="1-1"/>
 <wire x1="78.105" y1="2.54" x2="67.945" y2="2.54" width="0" layer="19" extent="1-1"/>
@@
 <signal name="N$34">
 <contactref element="U$3" pad="IN+"/>
-<contactref element="K3G3" pad="1"/>
+<contactref element="LIPO+" pad="1"/>
 <wire x1="-31.115" y1="-41.91" x2="32.46" y2="42.015" width="0" layer="19" extent="1-1"/>
 </signal>
+<signal name="N$35">
+<contactref element="U$4" pad="IN_L"/>
+<contactref element="AMP_IN_L" pad="1"/>
+<wire x1="75.565" y1="2.54" x2="-31.115" y2="-64.77" width="0" layer="19" extent="1-1"/>
+</signal>
+<signal name="N$36">
+<contactref element="U$4" pad="IN_R"/>
+<contactref element="AMP_IN_R" pad="1"/>
+<wire x1="80.645" y1="2.54" x2="-31.115" y2="-70.485" width="0" layer="19" extent="1-1"/>
+</signal>
+<signal name="N$37">
+<contactref element="U$4" pad="OUT_L_+"/>
+<contactref element="AMP_OUT_L_+" pad="1"/>
+<wire x1="60.325" y1="2.54" x2="-31.115" y2="-81.915" width="0" layer="19" extent="1-1"/>
+</signal>
+<signal name="N$38">
+<contactref element="U$4" pad="OUT_L_-"/>
+<contactref element="AMP_OUT_L_-" pad="1"/>
+<wire x1="62.865" y1="2.54" x2="-31.115" y2="-76.2" width="0" layer="19" extent="1-1"/>
+</signal>
+<signal name="N$39">
+<contactref element="U$4" pad="OUT_R_-"/>
+<contactref element="AMP_OUT_R_-" pad="1"/>
+<wire x1="55.245" y1="2.54" x2="-31.115" y2="-87.63" width="0" layer="19" extent="1-1"/>
+</signal>
+<signal name="N$40">
+<contactref element="U$4" pad="OUT_R_+"/>
+<contactref element="AMP_OUT_R_+" pad="1"/>
+<wire x1="57.785" y1="2.54" x2="-31.115" y2="-93.345" width="0" layer="19" extent="1-1"/>
+</signal>
 </signals>

Commit message: weiter gemacht
Parts:
- removed AMP_5V, AMP_GND, L+3, LB, LIPO+, LIPO-, MISC_5V, MISC_GND: (no value), wz:PIN-HEADER-1
- removed ZUM_PI: JST-XH_BUCHSE-4-, wz:JST-XH_BUCHSE-4
- added EXT_SCL_BUS, EXT_SDA_BUS, KEY_OFF_1, KEY_OFF_2, KEY_ON_1, KEY_ON_2: (no value), wz:PIN-HEADER-1
- added Q1: (no value), wz:TSSOP8-4.4MM
- added R17: 47k, wz:0603
- DISPLAY: device con-lstb:MA12-1 -> wz:PIN-HEADER-DISPLAY
- R1: value 100 -> (none)
- R3: value (none) -> 100k
- moved DISPLAY 141.0 mm to (-14.6, -99.1)
- moved R3 136.0 mm to (-31.1, -120.0), flipped to the top
- renumbered +5V to EXT_+5V, GND to EXT_GND, LG to L2, LR to L1
Connections:
- net LASER_G renamed LASER_2
- net N$1 renamed I_LED_R
- net N$10 renamed I_LED_B
- net N$17 renamed TX
- net N$2 renamed I_LED_G
- net N$26 renamed AMBI_LIGHT
- net N$3 renamed I_IR_TAKT_-
- net N$7 renamed I_LASER_2
- net N$8 renamed I_LED_W
- net N$9 renamed I_LASER_1
- removed net LASER_B: R3.1, ULN2803.13
- removed net LASER_R: R1.1, ULN2803.15
- removed net N$14: C5.2, IC1.25, R4.1, R5.2
- removed net N$19: LB.1, R3.2
- removed net N$27: R7.1, ZUM_PI.P$4
- removed net N$28: R6.1, ZUM_PI.P$3
- removed net N$34: LIPO+.1, U$3.IN+
- removed net N$4: IC1.12, ULN2803.4
- removed net SCL: BUS.P$4, D2.4, IC1.28, R7.2
- removed net SDA: BUS.P$3, D2.3, IC1.27, R6.2
- removed net V_BATT: B+.1, R4.2
- new net BACKLIGHT: DISPLAY.8, ULN2803.15
- new net BATT_+: B+.1, KEY_ON_2.1, R4.2, U$3.IN+
- new net BATT_-: B-.1, Q1.2, Q1.3, R3.2
- new net I_BACKLIGHT: PI.12, ULN2803.4
- new net LASER_1: R1.1, ULN2803.13
- new net N$1: DISPLAY.14, PI.13
- new net N$2: DISPLAY.11, PI.26
- new net N$26: KEY_ON_1.1, R17.1
- new net N$44: DISPLAY.1, PI.1
- new net N$45: DISPLAY.2, PI.9
- new net N$47: DISPLAY.5, PI.18
- new net N$48: DISPLAY.12, DISPLAY.6, PI.19
- new net N$49: DISPLAY.13, DISPLAY.9, PI.21
- new net N$50: DISPLAY.4, PI.22
- new net N$51: DISPLAY.10, DISPLAY.7, PI.23
- new net N$52: DISPLAY.3, PI.24
- new net ONOFF: IC1.32, KEY_OFF_1.1, Q1.4, R17.2, R3.1
- new net SCL_BUS: BUS.P$4, D2.4, EXT_SCL_BUS.1, IC1.28, R7.2
- new net SCL_PI: PI.5, R7.1
- new net SDA_BUS: BUS.P$3, D2.3, EXT_SDA_BUS.1, IC1.27, R6.2
- new net SDA_PI: PI.3, R6.1
- new net V_BATT_LOW: C5.1, IC1.25, R4.1, R5.2
- net +5V: now also PI.2, PI.4; no longer AMP_5V.1, MISC_5V.1, ZUM_PI.P$2
- net GND: now also C5.2, KEY_OFF_2.1, PI.6, Q1.1, Q1.8; no longer AMP_GND.1, B-.1, C5.1, LIPO-.1, MISC_GND.1, ZUM_PI.P$1
- net LASER_+: no longer L+3.1
Routing:
- net TX: track 30.4 -> 0.00 mm
- net SDA: track 19.5 -> 0.00 mm
- net +5V: track 89.9 -> 72.1 mm
- net SCL: track 16.2 -> 0.00 mm
- net N$14: track 6.55 -> 0.00 mm
- net LASER_B: track 5.33 -> 0.00 mm
- net I_LED_G: track 4.57 -> 0.00 mm
- net I_LED_B: track 4.43 -> 0.00 mm
- net I_IR_TAKT_-: track 4.37 -> 0.00 mm
- net LASER_R: track 4.28 -> 0.00 mm
- net I_LASER_1: track 4.24 -> 0.00 mm
- net N$4: track 4.06 -> 0.00 mm
- net I_LASER_2: track 4.02 -> 0.00 mm
- net N$28: track 3.59 -> 0.00 mm
- net N$27: track 3.59 -> 0.00 mm
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
Commit message: ...
Parts:
- removed Q1: (no value), wz:TSSOP8-4.4MM
- added R18: 10k, wz:0603
- added STEP_UP_ENABLE: (no value), wz:PIN-HEADER-1
- R17: value 47k -> 1k
- R3: value 100k -> 10k
- R5: value 10k -> 180k
Connections:
- removed net BATT_-: B-.1, Q1.2, Q1.3, R3.2
- net GND: now also B-.1, R3.2; no longer Q1.1, Q1.8
- net ONOFF: now also R18.1, R18.2, STEP_UP_ENABLE.1; no longer Q1.4
Changed lines of the file:
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@@
 </element>
 <element name="R4" library="wz" package="0603" value="120k" x="42.545" y="18.7325" rot="MR90"/>
-<element name="R5" library="wz" package="0603" value="10k" x="38.1" y="18.7325" rot="MR270"/>
+<element name="R5" library="wz" package="0603" value="180k" x="38.1" y="18.7325" rot="MR270"/>
 <element name="FUSE" library="resistor" package="L1812" value="PTC" x="10.795" y="31.115" rot="MR0"/>
 <element name="P-FET" library="zetex" package="SOT-23" value="" x="12.065" y="3.81" rot="MR90">
@@
 <element name="EXT_SCL_BUS" library="wz" package="PIN-HEADER-1" value="" x="-31.115" y="-106.045"/>
 <element name="EXT_SDA_BUS" library="wz" package="PIN-HEADER-1" value="" x="-31.115" y="-111.76"/>
-<element name="Q1" library="wz" package="TSSOP8-4.4MM" value="" x="-28.575" y="-115.57"/>
-<element name="R3" library="wz" package="0603" value="100k" x="-31.115" y="-120.015"/>
+<element name="R3" library="wz" package="0603" value="10k" x="-31.115" y="-120.015"/>
 <element name="KEY_ON_1" library="wz" package="PIN-HEADER-1" value="" x="-31.115" y="-126.365"/>
 <element name="KEY_ON_2" library="wz" package="PIN-HEADER-1" value="" x="-31.115" y="-132.08"/>
-<element name="R17" library="wz" package="0603" value="47k" x="-31.115" y="-136.525"/>
+<element name="R17" library="wz" package="0603" value="1k" x="-31.115" y="-136.525"/>
 <element name="KEY_OFF_1" library="wz" package="PIN-HEADER-1" value="" x="-31.115" y="-142.875"/>
 <element name="KEY_OFF_2" library="wz" package="PIN-HEADER-1" value="" x="-31.115" y="-148.59"/>
+<element name="STEP_UP_ENABLE" library="wz" package="PIN-HEADER-1" value="" x="-31.115" y="-154.305"/>
+<element name="R18" library="wz" package="0603" value="10k" x="-31.115" y="-158.75"/>
 </elements>
 <signals>
@@
 <contactref element="PI" pad="6"/>
 <contactref element="C5" pad="2"/>
-<contactref element="Q1" pad="1"/>
-<contactref element="Q1" pad="8"/>
 <contactref element="KEY_OFF_2" pad="1"/>
-<wire x1="-31.675" y1="-114.595" x2="-31.115" y2="-148.59" width="0" layer="19" extent="1-1"/>
-<wire x1="-25.475" y1="-114.595" x2="-31.675" y2="-114.595" width="0" layer="19" extent="1-1"/>
-<wire x1="2.225" y1="7.62" x2="-25.475" y2="-114.595" width="0" layer="19" extent="1-16"/>
+<contactref element="R3" pad="2"/>
+<contactref element="B-" pad="1"/>
+<wire x1="-30.265" y1="-120.015" x2="-31.115" y2="-148.59" width="0" layer="19" extent="1-1"/>
+<wire x1="2.225" y1="7.62" x2="-30.265" y2="-120.015" width="0" layer="19" extent="1-16"/>
 <wire x1="2.225" y1="17.78" x2="2.225" y2="7.62" width="0" layer="19" extent="16-16"/>
 <wire x1="2.225" y1="20.32" x2="2.225" y2="17.78" width="0" layer="19" extent="16-16"/>
@@
 <wire x1="38.735" y1="21.375" x2="36.83" y2="21.375" width="0" layer="19" extent="16-16"/>
 <wire x1="38.1" y1="19.5825" x2="38.735" y2="21.375" width="0" layer="19" extent="16-16"/>
+<wire x1="40.64" y1="22.225" x2="38.735" y2="21.375" width="0" layer="19" extent="16-16"/>
 <wire x1="40.005" y1="17.8825" x2="38.1" y2="19.5825" width="0" layer="19" extent="16-16"/>
 <wire x1="42.175" y1="14.9225" x2="40.005" y2="17.8825" width="0" layer="19" extent="16-16"/>
@@
 <wire x1="20.419" y1="30.33" x2="20.755" y2="30.33" width="0" layer="19" extent="16-16"/>
 <wire x1="21.493528125" y1="25.24983125" x2="20.755" y2="30.33" width="0" layer="19" extent="1-1"/>
-<wire x1="48.26" y1="22.225" x2="40.005" y2="17.8825" width="0" layer="19" extent="16-16"/>
+<wire x1="48.26" y1="22.225" x2="40.64" y2="22.225" width="0" layer="19" extent="1-1"/>
 <wire x1="48.26" y1="4.445" x2="42.175" y2="14.9225" width="0" layer="19" extent="16-16"/>
 <wire x1="67.945" y1="2.54" x2="48.26" y2="4.445" width="0" layer="19" extent="1-1"/>
@@
 <wire x1="16.725" y1="5.715" x2="36.0426" y2="13.24" width="0" layer="19" extent="16-16"/>
 </signal>
-<signal name="BATT_-">
-<contactref element="Q1" pad="2"/>
-<contactref element="Q1" pad="3"/>
-<contactref element="B-" pad="1"/>
-<contactref element="R3" pad="2"/>
-<wire x1="-31.675" y1="-115.895" x2="-30.265" y2="-120.015" width="0" layer="19" extent="1-1"/>
-<wire x1="-31.675" y1="-115.245" x2="-31.675" y2="-115.895" width="0" layer="19" extent="1-1"/>
-<wire x1="40.64" y1="22.225" x2="-31.675" y2="-115.245" width="0" layer="19" extent="1-1"/>
-</signal>
 <signal name="ONOFF">
 <contactref element="IC1" pad="32"/>
-<contactref element="Q1" pad="4"/>
 <contactref element="R3" pad="1"/>
 <contactref element="R17" pad="2"/>
 <contactref element="KEY_OFF_1" pad="1"/>
+<contactref element="STEP_UP_ENABLE" pad="1"/>
+<contactref element="R18" pad="2"/>
+<contactref element="R18" pad="1"/>
+<wire x1="-30.265" y1="-158.75" x2="-31.965" y2="-158.75" width="0" layer="19" extent="1-1"/>
+<wire x1="-31.115" y1="-154.305" x2="-31.965" y2="-158.75" width="0" layer="19" extent="1-1"/>
+<wire x1="-31.115" y1="-142.875" x2="-31.115" y2="-154.305" width="0" layer="19" extent="1-1"/>
 <wire x1="-30.265" y1="-136.525" x2="-31.115" y2="-142.875" width="0" layer="19" extent="1-1"/>
 <wire x1="-31.965" y1="-120.015" x2="-30.265" y2="-136.525" width="0" layer="19" extent="1-1"/>
-<wire x1="-31.675" y1="-116.545" x2="-31.965" y2="-120.015" width="0" layer="19" extent="1-1"/>
-<wire x1="36.0426" y1="12.44" x2="-31.675" y2="-116.545" width="0" layer="19" extent="1-16"/>
+<wire x1="36.0426" y1="12.44" x2="-31.965" y2="-120.015" width="0" layer="19" extent="1-16"/>
 </signal>
 <signal name="N$26">
