File: lasermodule/hardware/Lasermodul.brd (EAGLE design)
At the start: 51.7 x 35.5 mm, 89 parts, among them IC1 MEGA8-AI

Commit message: kleinere fixes lasermodul schaltplan
Parts:
- renumbered T5V to F_5V, TB to F_B, TG to F_G, TR to F_R, TW to F_W
Routing:
- net N$16: track 5.61 -> 0.00 mm
Changed lines of the file:
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@@
 <element name="L1+" library="wz" package="PIN-HEADER-1" value="" x="5.715" y="33.02" rot="R90"/>
 <element name="L2+" library="wz" package="PIN-HEADER-1" value="" x="5.715" y="30.48" rot="R90"/>
-<element name="TG" library="wz" package="PIN-HEADER-1" value="" x="5.715" y="20.32" rot="R90"/>
-<element name="TR" library="wz" package="PIN-HEADER-1" value="" x="5.715" y="22.86" rot="R90"/>
-<element name="TW" library="wz" package="PIN-HEADER-1" value="" x="5.715" y="7.62" rot="R90"/>
-<element name="TB" library="wz" package="PIN-HEADER-1" value="" x="5.715" y="17.78" rot="R90"/>
+<element name="F_G" library="wz" package="PIN-HEADER-1" value="" x="5.715" y="20.32" rot="R90"/>
+<element name="F_R" library="wz" package="PIN-HEADER-1" value="" x="5.715" y="22.86" rot="R90"/>
+<element name="F_W" library="wz" package="PIN-HEADER-1" value="" x="5.715" y="7.62" rot="R90"/>
+<element name="F_B" library="wz" package="PIN-HEADER-1" value="" x="5.715" y="17.78" rot="R90"/>
 <element name="IR_SNIPER_+" library="wz" package="PIN-HEADER-1" value="" x="5.715" y="2.54" rot="R90"/>
-<element name="T5V" library="wz" package="PIN-HEADER-1" value="" x="5.715" y="25.4" rot="R90"/>
+<element name="F_5V" library="wz" package="PIN-HEADER-1" value="" x="5.715" y="25.4" rot="R90"/>
 <element name="EXT_+5V" library="wz" package="PIN-HEADER-1" value="" x="45.72" y="22.225" rot="R180"/>
 <element name="IR_-_2" library="wz" package="PIN-HEADER-1" value="" x="5.715" y="5.08" rot="R90"/>
@@
 <signals>
 <signal name="+5V">
-<contactref element="T5V" pad="1"/>
+<contactref element="F_5V" pad="1"/>
 <contactref element="EXT_+5V" pad="1"/>
 <contactref element="LM1117" pad="3"/>
@@
 <wire x1="7.405" y1="12.7" x2="5.715" y2="12.7" width="0.4064" layer="16"/>
 </signal>
-<signal name="N$20">
-<contactref element="R14" pad="1"/>
-<contactref element="R14" pad="1"/>
-<contactref element="R8" pad="2"/>
-<contactref element="P-FET1" pad="3"/>
-<wire x1="16.725" y1="3.175" x2="15.025" y2="5.715" width="0.4064" layer="16"/>
-<wire x1="13.081" y1="4.8006" x2="14.6456" y2="4.8006" width="0.4064" layer="16"/>
-<wire x1="14.6456" y1="4.8006" x2="15.025" y2="5.715" width="0.4064" layer="16"/>
-</signal>
 <signal name="N$15">
 <contactref element="R10" pad="2"/>
-<contactref element="TR" pad="1"/>
+<contactref element="F_R" pad="1"/>
 <wire x1="5.715" y1="22.86" x2="6.67" y2="22.86" width="0.4064" layer="16"/>
 <wire x1="6.67" y1="22.86" x2="7.405" y2="22.225" width="0.4064" layer="16"/>
@@
 <signal name="N$21">
 <contactref element="R11" pad="2"/>
-<contactref element="TG" pad="1"/>
+<contactref element="F_G" pad="1"/>
 <wire x1="7.405" y1="20.32" x2="5.715" y2="20.32" width="0.4064" layer="16"/>
 <contactref element="C8" pad="2"/>
@@
 <signal name="N$22">
 <contactref element="R12" pad="2"/>
-<contactref element="TB" pad="1"/>
+<contactref element="F_B" pad="1"/>
 <wire x1="7.405" y1="17.78" x2="5.715" y2="17.78" width="0.4064" layer="16"/>
 <contactref element="C9" pad="2"/>
@@
 <signal name="N$23">
 <contactref element="R15" pad="2"/>
-<contactref element="TW" pad="1"/>
+<contactref element="F_W" pad="1"/>
 <wire x1="7.405" y1="7.62" x2="5.715" y2="7.62" width="0.4064" layer="16"/>
 <contactref element="C10" pad="2"/>
@@
 <wire x1="-30.4546" y1="-179.451" x2="-30.265" y2="-187.96" width="0" layer="19" extent="1-1"/>
 </signal>
-<signal name="N$46">
-<contactref element="R20" pad="1"/>
-<contactref element="R20" pad="1"/>
-<contactref element="P-FET2" pad="3"/>
-<contactref element="R19" pad="2"/>
-<wire x1="-27.52" y1="-182.88" x2="-30.265" y2="-182.88" width="0" layer="19" extent="1-1"/>
-<wire x1="-29.4894" y1="-177.419" x2="-30.265" y2="-182.88" width="0" layer="19" extent="1-1"/>
-</signal>
 <signal name="N$53">
 <contactref element="P-FET3" pad="1"/>
@@
 <wire x1="11.049" y1="3.8354" x2="-31.4198" y2="-177.419" width="0" layer="19" extent="1-16"/>
 </signal>
-<signal name="N$54">
+<signal name="I_IR_SHOTGUN">
+<contactref element="IC1" pad="26"/>
+<contactref element="R22" pad="1"/>
+<wire x1="36.0426" y1="17.24" x2="-31.965" y2="-200.025" width="0" layer="19" extent="1-16"/>
+</signal>
+<signal name="I_IR_SNIPER">
+<contactref element="IC1" pad="23"/>
+<contactref element="R19" pad="1"/>
+<wire x1="33.75" y1="19.5326" x2="-31.965" y2="-182.88" width="0" layer="19" extent="1-16"/>
+</signal>
+<signal name="IR_SNIPER_TX_+">
+<contactref element="R21" pad="1"/>
+<contactref element="IR_SNIPER_+" pad="1"/>
+<wire x1="5.715" y1="2.54" x2="-31.965" y2="-187.96" width="0" layer="19" extent="1-1"/>
+</signal>
+<signal name="N$16">
+<contactref element="R8" pad="2"/>
+<contactref element="P-FET1" pad="3"/>
+<contactref element="R14" pad="1"/>
+<contactref element="R14" pad="1"/>
+<wire x1="13.081" y1="4.8006" x2="15.025" y2="5.715" width="0" layer="19" extent="16-16"/>
+<wire x1="16.725" y1="3.175" x2="15.025" y2="5.715" width="0" layer="19" extent="16-16"/>
+</signal>
+<signal name="N$20">
+<contactref element="R20" pad="1"/>
+<contactref element="R20" pad="1"/>
+<contactref element="R19" pad="2"/>
+<contactref element="P-FET2" pad="3"/>
+<wire x1="-27.52" y1="-182.88" x2="-30.265" y2="-182.88" width="0" layer="19" extent="1-1"/>
+<wire x1="-29.4894" y1="-177.419" x2="-30.265" y2="-182.88" width="0" layer="19" extent="1-1"/>
+</signal>
+<signal name="N$55">
 <contactref element="R23" pad="1"/>
 <contactref element="R23" pad="1"/>
@@
 <wire x1="-29.4894" y1="-194.564" x2="-30.265" y2="-200.025" width="0" layer="19" extent="1-1"/>
 </signal>
-<signal name="I_IR_SHOTGUN">
-<contactref element="IC1" pad="26"/>
-<contactref element="R22" pad="1"/>
-<wire x1="36.0426" y1="17.24" x2="-31.965" y2="-200.025" width="0" layer="19" extent="1-16"/>
-</signal>
-<signal name="I_IR_SNIPER">
-<contactref element="IC1" pad="23"/>
-<contactref element="R19" pad="1"/>
-<wire x1="33.75" y1="19.5326" x2="-31.965" y2="-182.88" width="0" layer="19" extent="1-16"/>
-</signal>
-<signal name="IR_SNIPER_TX_+">
-<contactref element="R21" pad="1"/>
-<contactref element="IR_SNIPER_+" pad="1"/>
-<wire x1="5.715" y1="2.54" x2="-31.965" y2="-187.96" width="0" layer="19" extent="1-1"/>
-</signal>
 </signals>

Commit message: lasermodul: reverse polarity protection
Parts:
- removed FUSE: PTC, resistor:L1812
- removed ZD1: 5,6V, wz:Z-DIODE
- added P-FET4, P-FET5, P-FET6: (no value), zetex:SOT-23
- PI: device con-lstb:MA13-2 -> con-lstb:MA20-2
- moved PI 271.4 mm to (-6.99, -224.2)
- moved P-FET1 262.6 mm to (-30.5, -255.3), flipped to the top, turned to 0 degrees
- moved P-FET2 62.9 mm to (-30.5, -241.3)
- moved P-FET3 52.7 mm to (-30.5, -248.3)
Connections:
- removed net N$28: FUSE.1, U$3.OUT+
- new net N$46: P-FET4.2, PI.2, PI.4
- new net N$54: P-FET5.2, P-FET6.2, U$3.IN+
- net +3V2: now also P-FET1.2, P-FET2.1, P-FET3.1; no longer P-FET1.1, P-FET2.2, P-FET3.2
- net +3V3: now also P-FET1.1; no longer P-FET1.2
- net +5V: now also P-FET4.1, U$3.OUT+; no longer FUSE.2, PI.2, PI.4, ZD1.C
- net BATT_+: now also P-FET5.1, P-FET6.1; no longer U$3.IN+
- net GND: now also P-FET4.3, P-FET5.3, P-FET6.3; no longer ZD1.A
- net N$34: now also P-FET2.2; no longer P-FET2.1
- net N$53: now also P-FET3.2; no longer P-FET3.1
Routing:
- net +3V3: track 100.8 -> 98.4 mm

Commit message: another onoff
Parts:
- removed KEY_OFF_1, KEY_OFF_2, KEY_ON_1, KEY_ON_2, STEP_UP_ENABLE: (no value), wz:PIN-HEADER-1
- removed P-FET5, P-FET6: (no value), zetex:SOT-23
- removed R17: 1k, wz:0603
- removed R18, R3: 10k, wz:0603
- added OFF_1, OFF_2, ON_1, ON_2: (no value), wz:PIN-HEADER-1
- added OK1: SFH6186-2, optocoupler:SMD4-7
- added ON, REV: (no value), wz:TO252
- added R25: 270, wz:0603
- added R9: 10k, wz:0603
Connections:
- net IR_SHORGUN_TX_+ renamed IR_SHOTGUN_TX_+
- removed net N$26: KEY_ON_1.1, R17.1
- removed net N$54: P-FET5.2, P-FET6.2, U$3.IN+
- removed net STEPUP_EN: KEY_OFF_1.1, R17.2, R18.2, R3.1, STEP_UP_ENABLE.1
- new net BATT_-: REV.3
- new net N$28: ON.2, R9.1, REV.2
- new net ONOFF_2: OK1.3, ON.1, ON_2.1, R9.2
- net +3V3: now also R25.2
- net BATT_+: now also OK1.4, ON_1.1, REV.1, U$3.IN+; no longer KEY_ON_2.1, P-FET5.1, P-FET6.1
- net GND: now also OFF_1.1, OK1.2, ON.3; no longer KEY_OFF_2.1, P-FET5.3, P-FET6.3, R3.2
- net ONOFF: now also IC1.12, OFF_2.1, OK1.1, R25.1; no longer R18.1
