File: lasermodule/hardware/Lasermodul.brd (EAGLE design)
At the start: 51.7 x 35.5 mm, 89 parts, among them IC1 MEGA8-AI

Commit message: lasermodul routing started
Parts:
- removed AMP_OUT_L_+, AMP_OUT_L_-, AMP_OUT_R_+, AMP_OUT_R_-, EXT_+5V, EXT_GND, EXT_SCL_BUS, EXT_SDA_BUS, IR_-_1, IR_-_2, IR_SHOTGUN_+, IR_SNIPER_+: (no value), wz:PIN-HEADER-1
- removed P-FET4: (no value), zetex:SOT-23
- removed R1, R2: (no value), wz:0603
- added 2A_4A: PTC_FUSE, wz:PTC_FUSE_2920
- added AMP_IN_AGND, AMP_OUT_L+, AMP_OUT_L-, AMP_OUT_R+, AMP_OUT_R-, IR_SHOTGUN+, IR_SHOTGUN-, IR_SNIPER+, IR_SNIPER-: (no value), wz:PIN-HEADER-1
- added BUS1: JST-XH_BUCHSE-4-, wz:JST-XH_BUCHSE-4
- added C11: 4.7u, wz:0805
- added C12: 1000u, wz:C_UNIVERSAL
- added C13: 100n, wz:0603
- added D1(O): (no value), wz:DIODE_SMA_CLOSED
- added L1(O), L2(O): L, wz:L_5MM_CLOSED
- added R1(O), R2(O): (no value), wz:0603_CLOSED
- added R3(O): (no value), wz:0805_CLOSED
- BATT+, BATT-: device wz:PIN-HEADER-1 -> wz:PIN-HEADER-1_BIG
- moved ON_2 410.5 mm to (64.1, 57.1)
- moved OFF_2 410.3 mm to (37.5, 54.0)
- moved ON_1 402.8 mm to (64.1, 54.6)
- moved OFF_1 402.4 mm to (37.5, 51.4)
- moved R9 400.2 mm to (52.1, 67.3), flipped to the bottom, turned to 180 degrees
- moved R25 390.4 mm to (43.8, 54.6), flipped to the bottom, turned to 90 degrees
- moved ON 383.0 mm to (52.1, 72.4), flipped to the bottom
- moved OK1 381.0 mm to (54.6, 55.9), flipped to the bottom, turned to 90 degrees
- moved REV 380.1 mm to (41.9, 62.9), flipped to the bottom, turned to 180 degrees
- moved P-FET1 315.4 mm to (8.26, 57.8), flipped to the bottom
- moved P-FET3 314.8 mm to (12.7, 63.5), flipped to the bottom
- moved P-FET2 306.9 mm to (5.08, 63.5), flipped to the bottom
- moved R24 276.4 mm to (12.1, 67.9), flipped to the bottom, turned to 180 degrees
- moved PI 272.7 mm to (27.3, 46.4)
- moved R22 269.1 mm to (8.89, 66.0), flipped to the bottom, turned to 180 degrees
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- renumbered BUS to EXT_PORT, F_5V to FLASHL_5V, F_B to FLASHL_B, F_G to FLASHL_G, F_R to FLASHL_R, F_W to FLASHL_W, L1+ to LASER_1+, L1- to LASER_1-, L2+ to LASER_2+, L2- to LASER_2-
Connections:
- net +3V2 renamed EASTEREGG_NET
- net I_IR_TAKT_- renamed I_IR_CLK_-
- net I_LED_B renamed I_FLASHL_B
- net I_LED_G renamed I_FLASHL_G
- net I_LED_R renamed I_FLASHL_R
- net I_LED_W renamed I_FLASHL_W
- net LED_B renamed FLASHL_B
- net LED_G renamed FLASHL_G
- net LED_R renamed FLASHL_R
- net LED_W renamed FLASHL_W
- net N$1 renamed LCD_TOUCH_IRQ
- net N$2 renamed LCD_TOUCH_CS
- net N$35 renamed AMP_IN_L
- net N$36 renamed AMP_IN_R
- net N$47 renamed LCD_DC
- net N$48 renamed LCD_MOSI
- net N$49 renamed LCD_MISO
- net N$50 renamed LCD_RESET
- net N$51 renamed LCD_SCK
- net N$52 renamed LCD_CS
- net V_BATT_LOW renamed BATT+_ADC
- removed net BATT_+: BATT+.1, OK1.4, ON_1.1, R4.2, REV.1, U$3.IN+
- removed net BATT_-: REV.3
- removed net IR_TAKT_-: IR_-_1.1, IR_-_2.1, ULN2803.16
- removed net N$12: LASER_1-.1, R1.2
- removed net N$37: AMP_OUT_L_+.1, U$4.OUT_L_+
- removed net N$38: AMP_OUT_L_-.1, U$4.OUT_L_-
- removed net N$39: AMP_OUT_R_-.1, U$4.OUT_R_-
- removed net N$40: AMP_OUT_R_+.1, U$4.OUT_R_+
- new net AMP_IN_AGND: AMP_IN_AGND.1, U$4.AGND
- new net AMP_OUT_L+: AMP_OUT_L+.1, U$4.OUT_L_+
- new net AMP_OUT_L-: AMP_OUT_L-.1, U$4.OUT_L_-
- new net AMP_OUT_R+: AMP_OUT_R+.1, U$4.OUT_R_+
- new net AMP_OUT_R-: AMP_OUT_R-.1, U$4.OUT_R_-
- new net BATT+: 2A_4A.P$1, BATT+.1, R4.2
- new net BATT+_FUSE: 2A_4A.P$2, OK1.4, ON_1.1, REV.1, U$3.IN+
- new net BATT-: BATT-.1, REV.3
- new net IR_CLK_-: IR_SHOTGUN-.1, IR_SNIPER-.1, ULN2803.16
- new net LASER_1-: LASER_1-.1, R1(O).2
- new net LASER_2-: LASER_2-.1, R2(O).2
- new net N$27: L1(O).1, U$3.OUT+
- net +3V3: now also C11.1
- net +5V: now also BUS1.P$2, C12.1, C12.1B, D1(O).A, L1(O).2, R3(O).1; no longer EXT_+5V.1, P-FET4.1, U$3.OUT+, U$4.VCC
- net GND: now also BUS1.P$1, C11.2, C12.2, C12.2B, C13.1, DISPLAY.2, PI.14, PI.20, PI.25, PI.30, PI.34, PI.39, PI.9; no longer BATT-.1, EXT_GND.1, P-FET4.3, U$4.AGND
- net IR_SHOTGUN_TX_+: now also IR_SHOTGUN+.1; no longer IR_SHOTGUN_+.1
- net IR_SNIPER_TX_+: now also IR_SNIPER+.1; no longer IR_SNIPER_+.1
- net LASER_1: now also R1(O).1; no longer R1.1
- net LASER_2: now also R2(O).1; no longer R2.1
- net N$18: now also C13.2, IC1.20; no longer LASER_2-.1, R2.2
- net N$44: now also D1(O).C, PI.2, PI.4; no longer PI.1
- net N$45: now also L2(O).2, R3(O).2; no longer DISPLAY.2, PI.9
- net N$46: now also L2(O).1, U$4.VCC; no longer P-FET4.2, PI.2, PI.4
- net SCL_BUS: now also BUS1.P$4; no longer EXT_SCL_BUS.1
- net SDA_BUS: now also BUS1.P$3; no longer EXT_SDA_BUS.1
Routing:
- net IR_TAKT_-: track 27.0 -> 0.00 mm
- net IR_CLK_-: track 0.00 -> 25.8 mm
- net +3V3: track 98.4 -> 92.8 mm
- net +5V: track 69.0 -> 65.2 mm
- net BATT_+: track 2.75 -> 0.00 mm
- net N$18: track 1.69 -> 0.00 mm
- net N$12: track 1.69 -> 0.00 mm
- net LASER_2-: track 0.00 -> 1.69 mm
- net LASER_1-: track 0.00 -> 1.69 mm
- removed copper zone on layer 16, net N$5
- removed copper zone on layer 16, net N$6
Other:
- board size 51.7 x 35.5 mm -> 51.7 x 34.9 mm

Commit message: lots of bugs fixed
Parts:
- 2A_4A: value PTC_FUSE -> PTC_FUSEPTC_FUSE_2920_UNIVERSAL; device wz:PTC_FUSE_2920 -> wz:PTC_FUSE_2920_UNIVERSAL
- moved C12 68.1 mm to (56.5, 5.08), turned to 270 degrees
- moved C3 66.1 mm to (66.7, 5.08), turned to 270 degrees
- moved AMP_OUT_R- 41.9 mm to (97.2, 1.27)
- moved AMP_OUT_R+ 36.9 mm to (94.6, 1.27)
- moved AMP_OUT_L+ 31.8 mm to (92.1, 1.27)
- moved L1(O) 29.4 mm to (55.9, 19.1), turned to 270 degrees
- moved AMP_OUT_L- 26.7 mm to (89.5, 1.27)
- moved U$4 24.4 mm to (70.5, 22.9), turned to 0 degrees
- moved R3(O) 14.1 mm to (61.0, 19.1), turned to 180 degrees
- moved L2(O) 13.1 mm to (66.0, 19.1), turned to 180 degrees
- moved AMP_IN_R 8.98 mm to (71.8, 1.27)
- moved AMP_IN_AGND 4.02 mm to (74.3, 1.27)
- moved AMP_IN_L 1.80 mm to (76.8, 1.27)
- moved C2 1.42 mm to (82.5, 71.1)
- moved U$3 1.27 mm to (53.3, 23.5)
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
Commit message: was wieder raus genommen
Parts:
- moved AMP_IN_L 1.27 mm to (78.1, 1.27)
- moved AMP_IN_R 1.27 mm to (73.0, 1.27)
- moved AMP_OUT_L- 1.27 mm to (90.8, 1.27)
- moved AMP_OUT_R+ 1.27 mm to (95.9, 1.27)
- moved AMP_IN_AGND 1.27 mm to (75.6, 1.27)
- moved AMP_OUT_L+ 1.27 mm to (93.3, 1.27)
- moved AMP_OUT_R- 1.27 mm to (98.4, 1.27)
- moved U$4 1.27 mm to (71.8, 22.9)
Changed lines of the file:
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@@
 <element name="U$3" library="wz" package="XL6009-STEPUP-BOARD" value="XL6009-STEPUP-BOARD" x="53.34" y="23.495"/>
 <element name="U$2" library="wz" package="PI2" value="" x="80.01" y="-6.35"/>
-<element name="U$4" library="wz" package="PAM8403-AMP-BOARD" value="PAM8403-AMP-BOARD" x="70.485" y="22.86"/>
-<element name="AMP_IN_L" library="wz" package="PIN-HEADER-1" value="" x="76.835" y="1.27"/>
-<element name="AMP_IN_R" library="wz" package="PIN-HEADER-1" value="" x="71.755" y="1.27"/>
-<element name="AMP_OUT_L-" library="wz" package="PIN-HEADER-1" value="" x="89.535" y="1.27"/>
-<element name="AMP_OUT_L+" library="wz" package="PIN-HEADER-1" value="" x="92.075" y="1.27"/>
-<element name="AMP_OUT_R-" library="wz" package="PIN-HEADER-1" value="" x="97.155" y="1.27"/>
-<element name="AMP_OUT_R+" library="wz" package="PIN-HEADER-1" value="" x="94.615" y="1.27"/>
+<element name="U$4" library="wz" package="PAM8403-AMP-BOARD" value="PAM8403-AMP-BOARD" x="71.755" y="22.86"/>
+<element name="AMP_IN_L" library="wz" package="PIN-HEADER-1" value="" x="78.105" y="1.27"/>
+<element name="AMP_IN_R" library="wz" package="PIN-HEADER-1" value="" x="73.025" y="1.27"/>
+<element name="AMP_OUT_L-" library="wz" package="PIN-HEADER-1" value="" x="90.805" y="1.27"/>
+<element name="AMP_OUT_L+" library="wz" package="PIN-HEADER-1" value="" x="93.345" y="1.27"/>
+<element name="AMP_OUT_R-" library="wz" package="PIN-HEADER-1" value="" x="98.425" y="1.27"/>
+<element name="AMP_OUT_R+" library="wz" package="PIN-HEADER-1" value="" x="95.885" y="1.27"/>
 <element name="DISPLAY" library="wz" package="PIN-HEADER-DISPLAY" value="" x="19.685" y="39.37">
 <attribute name="MF" value="" x="19.685" y="39.37" size="1.778" layer="27" display="off"/>
@@
 <element name="L2(O)" library="wz" package="L_5MM_CLOSED" value="L" x="66.04" y="19.05" rot="R180"/>
 <element name="R3(O)" library="wz" package="0805_CLOSED" value="" x="60.96" y="19.05" rot="MR180"/>
-<element name="AMP_IN_AGND" library="wz" package="PIN-HEADER-1" value="" x="74.295" y="1.27"/>
+<element name="AMP_IN_AGND" library="wz" package="PIN-HEADER-1" value="" x="75.565" y="1.27"/>
 <element name="C13" library="wz" package="0603" value="100n" x="32.385" y="20.955" rot="MR0"/>
 <element name="2A_4A" library="wz" package="PTC_FUSE_2920_UNIVERSAL" value="PTC_FUSEPTC_FUSE_2920_UNIVERSAL" x="27.305" y="67.945" rot="MR180"/>
@@
 <wire x1="56.515" y1="7.62" x2="55.88" y2="16.55" width="0" layer="19" extent="1-1"/>
 <wire x1="56.515" y1="7.284" x2="56.515" y2="7.62" width="0" layer="19" extent="16-16"/>
-<wire x1="66.675" y1="7.62" x2="56.515" y2="7.62" width="0" layer="19" extent="1-1"/>
-<wire x1="66.675" y1="7.284" x2="66.675" y2="7.62" width="0" layer="19" extent="16-16"/>
-<wire x1="45.72" y1="11.43" x2="55.88" y2="16.55" width="0" layer="19" extent="1-1"/>
-<wire x1="45.72" y1="4.445" x2="45.72" y2="11.43" width="0" layer="19" extent="1-1"/>
-<wire x1="45.72" y1="22.5425" x2="45.72" y2="11.43" width="0" layer="19" extent="16-16"/>
+<wire x1="49.53" y1="24.4475" x2="55.88" y2="16.55" width="0" layer="19" extent="16-16"/>
 <wire x1="15.725" y1="30.33" x2="17.53" y2="31.75" width="0" layer="19" extent="16-16"/>
 <wire x1="5.715" y1="30.48" x2="5.715" y2="25.4" width="0" layer="19" extent="1-1"/>
 <wire x1="5.715" y1="33.02" x2="5.715" y2="30.48" width="0" layer="19" extent="1-1"/>
+<wire x1="66.675" y1="7.62" x2="56.515" y2="7.62" width="0" layer="19" extent="1-1"/>
+<wire x1="66.675" y1="7.284" x2="66.675" y2="7.62" width="0" layer="19" extent="16-16"/>
+<wire x1="45.72" y1="11.43" x2="45.72" y2="22.5425" width="0" layer="19" extent="16-16"/>
+<wire x1="45.72" y1="4.445" x2="45.72" y2="11.43" width="0" layer="19" extent="1-1"/>
 <wire x1="5.08" y1="54.905" x2="5.715" y2="33.02" width="0" layer="19" extent="16-16"/>
 </signal>
@@
 <contactref element="U$4" pad="IN_L"/>
 <contactref element="AMP_IN_L" pad="1"/>
-<wire x1="76.835" y1="1.27" x2="76.835" y2="21.59" width="0" layer="19" extent="1-1"/>
+<wire x1="78.105" y1="1.27" x2="78.105" y2="21.59" width="0" layer="19" extent="1-1"/>
 </signal>
 <signal name="AMP_IN_R">
 <contactref element="U$4" pad="IN_R"/>
 <contactref element="AMP_IN_R" pad="1"/>
-<wire x1="71.755" y1="1.27" x2="71.755" y2="21.59" width="0" layer="19" extent="1-1"/>
+<wire x1="73.025" y1="1.27" x2="73.025" y2="21.59" width="0" layer="19" extent="1-1"/>
 </signal>
 <signal name="AMP_OUT_L+">
 <contactref element="U$4" pad="OUT_L_+"/>
 <contactref element="AMP_OUT_L+" pad="1"/>
-<wire x1="92.075" y1="1.27" x2="92.075" y2="21.59" width="0" layer="19" extent="1-1"/>
+<wire x1="93.345" y1="1.27" x2="93.345" y2="21.59" width="0" layer="19" extent="1-1"/>
 </signal>
 <signal name="AMP_OUT_L-">
 <contactref element="U$4" pad="OUT_L_-"/>
 <contactref element="AMP_OUT_L-" pad="1"/>
-<wire x1="89.535" y1="1.27" x2="89.535" y2="21.59" width="0" layer="19" extent="1-1"/>
+<wire x1="90.805" y1="1.27" x2="90.805" y2="21.59" width="0" layer="19" extent="1-1"/>
 </signal>
 <signal name="AMP_OUT_R-">
 <contactref element="U$4" pad="OUT_R_-"/>
 <contactref element="AMP_OUT_R-" pad="1"/>
-<wire x1="97.155" y1="1.27" x2="97.155" y2="21.59" width="0" layer="19" extent="1-1"/>
+<wire x1="98.425" y1="1.27" x2="98.425" y2="21.59" width="0" layer="19" extent="1-1"/>
 </signal>
 <signal name="AMP_OUT_R+">
 <contactref element="U$4" pad="OUT_R_+"/>
 <contactref element="AMP_OUT_R+" pad="1"/>
-<wire x1="94.615" y1="1.27" x2="94.615" y2="21.59" width="0" layer="19" extent="1-1"/>
+<wire x1="95.885" y1="1.27" x2="95.885" y2="21.59" width="0" layer="19" extent="1-1"/>
 </signal>
 <signal name="LCD_DC">
@@
 <contactref element="L2(O)" pad="1"/>
 <contactref element="U$4" pad="VCC"/>
-<wire x1="68.54" y1="19.05" x2="81.915" y2="21.59" width="0" layer="19" extent="1-1"/>
+<wire x1="68.54" y1="19.05" x2="83.185" y2="21.59" width="0" layer="19" extent="1-1"/>
 </signal>
 <signal name="AMP_IN_AGND">
 <contactref element="AMP_IN_AGND" pad="1"/>
 <contactref element="U$4" pad="AGND"/>
-<wire x1="74.295" y1="1.27" x2="74.295" y2="21.59" width="0" layer="19" extent="1-1"/>
+<wire x1="75.565" y1="1.27" x2="75.565" y2="21.59" width="0" layer="19" extent="1-1"/>
 </signal>
 <signal name="BATT+_ADC">

Commit message: lasermodul routing
Parts:
- moved BATT+ 98.5 mm to (97.2, 2.54)
- moved 2A_4A 92.0 mm to (97.8, 8.89), turned to 0 degrees
- moved R4 84.8 mm to (98.4, 14.3), turned to 270 degrees
- moved C5 79.2 mm to (94.6, 14.3), turned to 270 degrees
- moved AMP_IN_AGND 73.3 mm to (5.08, 21.3)
- moved AMP_IN_L 73.3 mm to (7.62, 21.3)
- moved AMP_IN_R 73.3 mm to (2.54, 21.3)
- moved BATT- 73.3 mm to (97.2, 19.7)
- moved AMP_OUT_L- 71.9 mm to (20.3, 15.6)
- moved AMP_OUT_R+ 71.9 mm to (25.4, 15.6)
- moved AMP_OUT_L+ 71.9 mm to (22.9, 15.6)
- moved AMP_OUT_R- 71.9 mm to (27.9, 15.6)
- moved U$4 70.5 mm to (1.27, 20.0)
- moved LOGO1 68.2 mm to (59.1, 75.6)
- moved REV 63.4 mm to (95.2, 28.6)
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Connections:
- net BACKLIGHT: now also ULN2803.18; no longer ULN2803.15
- net FLASHL_G: now also ULN2803.16; no longer ULN2803.17
- net FLASHL_R: now also ULN2803.17; no longer ULN2803.18
- net IR_CLK_-: now also ULN2803.15; no longer ULN2803.16
- net I_BACKLIGHT: now also ULN2803.1; no longer ULN2803.4
- net I_FLASHL_G: now also ULN2803.3; no longer ULN2803.2
- net I_FLASHL_R: now also ULN2803.2; no longer ULN2803.1
- net I_IR_CLK_-: now also ULN2803.4; no longer ULN2803.3
- net SCL_BUS: now also D2.3; no longer D2.4
- net SDA_BUS: now also D2.4; no longer D2.3
Routing:
- net +3V3: track 92.8 -> 32.9 mm
- net BATT+_ADC: track 0.00 -> 54.3 mm, vias 0 -> 2
- net BATT+_FUSE: track 0.00 -> 53.7 mm
- net ONOFF: track 0.00 -> 47.9 mm, vias 0 -> 2
- net RESET: track 57.0 -> 18.9 mm, vias 0 -> 1
- net RX: track 27.8 -> 0.00 mm
- net LCD_MISO: track 0.00 -> 26.7 mm
- net LCD_TOUCH_CS: track 0.00 -> 26.2 mm
- net IR_CLK_-: track 25.8 -> 0.00 mm
- net LCD_MOSI: track 0.00 -> 24.4 mm
- net N$46: track 0.00 -> 23.4 mm
- net LCD_SCK: track 0.00 -> 22.5 mm
- net ONOFF_2: track 0.00 -> 22.0 mm
- net +5V: track 65.2 -> 86.6 mm
- net LCD_TOUCH_IRQ: track 0.00 -> 16.6 mm
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- added copper zone on layer 1, net GND
- removed copper zone on layer 16, net +3V3
- removed copper zone on layer 16, net N$29
Other:
- board outline removed

Commit message: routing
Parts:
- moved C11 45.5 mm to (58.7, 22.9), turned to 180 degrees
- moved R22 25.7 mm to (59.7, 60.0)
- moved C2 23.2 mm to (67.0, 43.5), turned to 180 degrees
- moved LASER_1- 10.2 mm to (21.9, 24.8)
- moved R6 6.68 mm to (32.1, 36.2)
- moved R7 5.43 mm to (32.1, 34.0)
- moved LASER_2- 5.12 mm to (21.9, 27.0)
- moved LASER_1+ 4.18 mm to (11.4, 22.2)
- moved LASER_2+ 3.84 mm to (8.57, 29.2)
- moved R2(O) 1.93 mm to (25.7, 26.4)
- moved R1(O) 1.91 mm to (25.7, 24.8)
Routing:
- net +3V3: track 32.9 -> 103.6 mm, vias 0 -> 2
- net N$44: track 0.00 -> 53.5 mm
- net +5V: track 86.6 -> 139.6 mm
- net RX: track 0.00 -> 42.1 mm, vias 0 -> 1
- net I_BACKLIGHT: track 0.00 -> 38.6 mm, vias 0 -> 1
- net IR_CLK_-: track 0.00 -> 35.6 mm, vias 0 -> 1
- net SCL_PI: track 0.00 -> 33.5 mm, vias 0 -> 1
- net SDA_BUS: track 12.9 -> 43.6 mm, vias 0 -> 2
- net SCL_BUS: track 13.0 -> 42.3 mm, vias 0 -> 2
- net SDA_PI: track 0.00 -> 24.8 mm, vias 0 -> 1
- net AMBI_LIGHT: track 4.74 -> 12.4 mm
- net GND: track 0.00 -> 3.67 mm
- net KEY_3: track 9.03 -> 10.1 mm

Commit message: routing
Parts:
- added H1, H2: MOUNT-PAD-ROUND3.0, holes:3,0-PAD
- moved R22 60.5 mm to (6.67, 30.8), turned to 0 degrees
- moved R23 51.7 mm to (6.67, 32.7), turned to 180 degrees
- moved R21 49.8 mm to (4.45, 28.3), turned to 90 degrees
- moved R20 47.9 mm to (6.67, 25.4)
- moved P-FET3 46.5 mm to (6.67, 35.2), turned to 270 degrees
- moved P-FET2 46.1 mm to (6.67, 28.3), turned to 270 degrees
- moved R24 44.8 mm to (4.45, 35.2), turned to 90 degrees
- moved C5 44.8 mm to (52.7, 30.2), turned to 180 degrees
- moved R14 42.4 mm to (10.2, 25.4), turned to 180 degrees
- moved P-FET1 41.3 mm to (9.84, 28.3), turned to 270 degrees
- moved R8 39.8 mm to (10.2, 23.5), turned to 0 degrees
- moved R19 39.3 mm to (6.67, 23.5), turned to 0 degrees
- moved C2 34.4 mm to (49.8, 13.7)
- moved U$1 34.2 mm to (35.6, 36.2)
- moved C1 15.5 mm to (34.3, 33.7)
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Routing:
- net RX: track 42.1 -> 0.00 mm, vias 1 -> 0
- net +5V: track 139.6 -> 117.6 mm
- net +3V3: track 103.6 -> 84.1 mm, vias 2 -> 1
- net ONOFF: track 47.8 -> 66.4 mm
- net RESET: track 19.3 -> 3.74 mm, vias 1 -> 0
- net KEY_3: track 10.1 -> 0.00 mm, vias 1 -> 0
- net AMBI_LIGHT: track 12.4 -> 22.3 mm
- net KEY_1: track 8.90 -> 0.00 mm
- net KEY_2: track 7.12 -> 0.00 mm
- net BATT+_ADC: track 54.3 -> 60.7 mm
- net I_FLASHL_G: track 9.01 -> 2.75 mm
- net I_FLASHL_W: track 19.1 -> 12.8 mm
- net I_FLASHL_B: track 9.19 -> 3.16 mm
- net I_LASER_2: track 8.80 -> 2.77 mm
- net I_LASER_1: track 9.00 -> 2.97 mm
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Other:
- board text added: "Meow"
