File: lasermodule/hardware/lasermodule.brd (EAGLE design)
At the start: 76.8 x 49.5 mm, 88 parts, among them IC1 MEGA8-AI

Commit message: routing
Parts:
- added LOGO2: OSHW-LOGOM, SparkFun-Aesthetics:OSHW-LOGO-M
Other:
- board text added: "Lasertag Lasermodule v1.0 warpzone.ms"
- board text removed: "Lasertag Weapon v1.0 warpzone.ms"
Changed lines of the file:
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@@
 <grid distance="0.635" unitdist="mm" unit="mm" style="dots" multiple="1" display="yes" altdistance="0.15875" altunitdist="mm" altunit="mm"/>
 <layers>
-<layer number="1" name="Top" color="4" fill="1" visible="no" active="yes"/>
+<layer number="1" name="Top" color="4" fill="1" visible="yes" active="yes"/>
 <layer number="16" name="Bottom" color="1" fill="1" visible="yes" active="yes"/>
 <layer number="17" name="Pads" color="2" fill="1" visible="yes" active="yes"/>
@@
 <text x="66.675" y="3.81" size="1.27" layer="26" font="vector" ratio="10" rot="MR0" align="bottom-right">ON_2</text>
 <text x="66.675" y="1.27" size="1.27" layer="26" font="vector" ratio="10" rot="MR0" align="bottom-right">ON_1</text>
-<text x="29.845" y="30.7975" size="1.016" layer="25" font="vector" ratio="10" rot="R270">GND</text>
+<text x="29.845" y="30.7975" size="0.6096" layer="25" font="vector" ratio="10" rot="R270">GND</text>
 <text x="32.385" y="31.75" size="1.016" layer="25" font="vector" ratio="10" rot="R270">5V</text>
 <text x="27.305" y="31.75" size="1.016" layer="25" font="vector" ratio="10" rot="R270">RX</text>
@@
 <text x="42.545" y="34.6075" size="1.27" layer="25" font="vector" ratio="10" rot="R270">SCK</text>
 <text x="45.085" y="12.54125" size="1.27" layer="25" font="vector" ratio="10">L_PWR</text>
-<text x="26.82875" y="22.225" size="1.27" layer="25" font="vector" ratio="10">Lasertag Weapon
+<text x="26.82875" y="21.9075" size="1.27" layer="25" font="vector" ratio="10">Lasertag
+Lasermodule
 v1.0
 warpzone.ms</text>
@@
 <attribute name="VALUE" x="19.05" y="15.24" size="1.27" layer="28" rot="MR270"/>
 </element>
+<element name="LOGO2" library="SparkFun-Aesthetics" package="OSHW-LOGO-M" value="OSHW-LOGOM" x="64.77" y="24.28875" rot="MR0"/>
 </elements>
 <signals>
